Commit message: moveit config and bringup

File: my_robot_description/urdf/gripper.xacro (robot description, xacro)
@@ -1,53 +1,47 @@
 <?xml version="1.0"?>
-<robot name="temp" xmlns:xacro="http://www.ros.org/wiki/xacro">
-    <material name="dark_green">
-        <color rgba="0 0.4 0.0 1"/>
-    </material>
-    <material name="dark_green">
-        <color rgba="0 0.6 0.0 1"/>
-    </material>
+<robot xmlns:xacro="http://www.ros.org/wiki/xacro">
     <link name="gripper_base_link">
         <visual>
-            <origin xyz="0 0 0.01" rpy="0 0 0" />
             <geometry>
                 <box size="0.2 0.06 0.02" />
             </geometry>
+            <origin xyz="0 0 0.01" rpy="0 0 0" />
             <material name="dark_green" />
         </visual>
         <collision>
-            <origin xyz="0 0 0.01" rpy="0 0 0" />
             <geometry>
                 <box size="0.2 0.06 0.02" />
             </geometry>
+            <origin xyz="0 0 0.01" rpy="0 0 0" />
         </collision>
     </link>
     <link name="gripper_left_finger_link">
         <visual>
-            <origin xyz="0 0 0.04" rpy="0 0 0" />
             <geometry>
                 <box size="0.02 0.06 0.08" />
             </geometry>
+            <origin xyz="0 0 0.04" rpy="0 0 0" />
             <material name="light_green" />
         </visual>
         <collision>
-            <origin xyz="0 0 0.04" rpy="0 0 0" />
             <geometry>
                 <box size="0.02 0.06 0.08" />
             </geometry>
+            <origin xyz="0 0 0.04" rpy="0 0 0" />
         </collision>
     </link>
     <link name="gripper_right_finger_link">
         <visual>
-            <origin xyz="0 0 0.04" rpy="0 0 0" />
             <geometry>
                 <box size="0.02 0.06 0.08" />
             </geometry>
+            <origin xyz="0 0 0.04" rpy="0 0 0" />
             <material name="light_green" />
         </visual>
         <collision>
-            <origin xyz="0 0 0.04" rpy="0 0 0" />
             <geometry>
                 <box size="0.02 0.06 0.08" />
             </geometry>
+            <origin xyz="0 0 0.04" rpy="0 0 0" />
         </collision>
     </link>

File: my_robot_description/urdf/my_robot.urdf.xacro (robot description, xacro)
@@ -3,3 +3,10 @@
     <xacro:include filename="common_properties.xacro" />
     <xacro:include filename="arm.xacro" />
+    <xacro:include filename="gripper.xacro" />
+    <xacro:include filename="my_robot.ros2_control.xacro" />
+    <joint name="gripper_base_joint" type="fixed">
+        <parent link="tool_link" />
+        <child link="gripper_base_link" />
+        <origin xyz="0 0 0" rpy="0 0 0" />
+    </joint>
 </robot>
